File: Hardware/OpenBook.sch (EAGLE design)
At the start: 103 parts, among them IC1 XC6220A331MR-G, IC2 BD5229G-TR, J1 SAMACSYS_PARTS_USB4110-GF-A, J2 112A-TAAR-R03_ATTEND, J3 FH34SRJ-24S-0.5SH_99_, J4 QWIIC_RIGHT_ANGLE, Q1 20V/4.2A/52mΩ/1.4W, Q2 SI1308EDL-T1-GE3, Q3 20V/4.2A/52mΩ/1.4W, U1 ESP32_WROVER_SPARKFUN-IC-POWE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

Commit message: Fixed shorted GND on PIN21
Signed-off-by: Bicoiu Ionut <159699747+bicoiu@users.noreply.github.com>
Connections:
- net GND: no longer C11.2, C12.2, C13.2, C14.2, C15.2, C16.2, C17.2, C18.2
- net PREVGH: now also C11.2, C12.2, C13.2, C14.2, C15.2, C16.2, C17.2, C18.2
Changed lines of the file:
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@@
 <text x="154.94" y="139.7" size="2.54" layer="95">Display Type Selector
 </text>
-<text x="-162.56" y="142.24" size="2.54" layer="91">E-Paper Drive Circuit</text>
+<text x="-162.56" y="142.24" size="2.54" layer="95">E-Paper Drive Circuit</text>
 <text x="-40.64" y="142.24" size="2.54" layer="95">Li-Po Battery Charging Controller</text>
 <text x="60.96" y="139.7" size="2.54" layer="95">ESP32 C6
@@
 <pinref part="SUPPLY60" gate="G$1" pin="GND"/>
 </segment>
-<segment>
-<pinref part="C11" gate="G$1" pin="2"/>
-<wire x1="-162.56" y1="63.5" x2="-165.1" y2="63.5" width="0.1524" layer="91"/>
-<wire x1="-165.1" y1="63.5" x2="-165.1" y2="71.12" width="0.1524" layer="91"/>
-<pinref part="C12" gate="G$1" pin="2"/>
-<wire x1="-149.86" y1="60.96" x2="-165.1" y2="60.96" width="0.1524" layer="91"/>
-<wire x1="-165.1" y1="60.96" x2="-165.1" y2="63.5" width="0.1524" layer="91"/>
-<pinref part="C13" gate="G$1" pin="2"/>
-<wire x1="-137.16" y1="58.42" x2="-165.1" y2="58.42" width="0.1524" layer="91"/>
-<wire x1="-165.1" y1="58.42" x2="-165.1" y2="60.96" width="0.1524" layer="91"/>
-<pinref part="C14" gate="G$1" pin="2"/>
-<wire x1="-124.46" y1="55.88" x2="-139.7" y2="55.88" width="0.1524" layer="91"/>
-<wire x1="-139.7" y1="55.88" x2="-165.1" y2="55.88" width="0.1524" layer="91"/>
-<wire x1="-165.1" y1="55.88" x2="-165.1" y2="58.42" width="0.1524" layer="91"/>
-<pinref part="C15" gate="G$1" pin="2"/>
-<wire x1="-137.16" y1="53.34" x2="-165.1" y2="53.34" width="0.1524" layer="91"/>
-<wire x1="-165.1" y1="53.34" x2="-165.1" y2="55.88" width="0.1524" layer="91"/>
-<pinref part="C16" gate="G$1" pin="2"/>
-<wire x1="-149.86" y1="50.8" x2="-165.1" y2="50.8" width="0.1524" layer="91"/>
-<wire x1="-165.1" y1="50.8" x2="-165.1" y2="53.34" width="0.1524" layer="91"/>
-<wire x1="-165.1" y1="50.8" x2="-165.1" y2="48.26" width="0.1524" layer="91"/>
-<wire x1="-165.1" y1="48.26" x2="-165.1" y2="40.64" width="0.1524" layer="91"/>
-<wire x1="-165.1" y1="40.64" x2="-154.94" y2="40.64" width="0.1524" layer="91"/>
-<pinref part="C18" gate="G$1" pin="2"/>
-<wire x1="-139.7" y1="55.88" x2="-139.7" y2="71.12" width="0.1524" layer="91"/>
-<label x="-139.7" y="71.12" size="1.4224" layer="95" rot="R90" xref="yes"/>
-<pinref part="C17" gate="G$1" pin="2"/>
-<wire x1="-162.56" y1="48.26" x2="-165.1" y2="48.26" width="0.1524" layer="91"/>
-<junction x="-165.1" y="63.5"/>
-<junction x="-165.1" y="60.96"/>
-<junction x="-165.1" y="58.42"/>
-<junction x="-139.7" y="55.88"/>
-<junction x="-165.1" y="55.88"/>
-<junction x="-165.1" y="53.34"/>
-<junction x="-165.1" y="50.8"/>
-<junction x="-165.1" y="48.26"/>
-<pinref part="GND1" gate="1" pin="GND"/>
-</segment>
 </net>
 <net name="N$1" class="0">
@@
 <label x="-106.68" y="96.52" size="2.54" layer="95" xref="yes"/>
 </segment>
-</net>
+<segment>
+<pinref part="C11" gate="G$1" pin="2"/>
+<wire x1="-162.56" y1="63.5" x2="-165.1" y2="63.5" width="0.1524" layer="91"/>
+<wire x1="-165.1" y1="63.5" x2="-165.1" y2="71.12" width="0.1524" layer="91"/>
+<pinref part="C12" gate="G$1" pin="2"/>
+<wire x1="-149.86" y1="60.96" x2="-165.1" y2="60.96" width="0.1524" layer="91"/>
+<wire x1="-165.1" y1="60.96" x2="-165.1" y2="63.5" width="0.1524" layer="91"/>
+<pinref part="C13" gate="G$1" pin="2"/>
+<wire x1="-137.16" y1="58.42" x2="-144.78" y2="58.42" width="0.1524" layer="91"/>
+<wire x1="-144.78" y1="58.42" x2="-165.1" y2="58.42" width="0.1524" layer="91"/>
+<wire x1="-165.1" y1="58.42" x2="-165.1" y2="60.96" width="0.1524" layer="91"/>
+<pinref part="C14" gate="G$1" pin="2"/>
+<wire x1="-124.46" y1="55.88" x2="-165.1" y2="55.88" width="0.1524" layer="91"/>
+<wire x1="-165.1" y1="55.88" x2="-165.1" y2="58.42" width="0.1524" layer="91"/>
+<pinref part="C15" gate="G$1" pin="2"/>
+<wire x1="-137.16" y1="53.34" x2="-165.1" y2="53.34" width="0.1524" layer="91"/>
+<wire x1="-165.1" y1="53.34" x2="-165.1" y2="55.88" width="0.1524" layer="91"/>
+<pinref part="C16" gate="G$1" pin="2"/>
+<wire x1="-149.86" y1="50.8" x2="-165.1" y2="50.8" width="0.1524" layer="91"/>
+<wire x1="-165.1" y1="50.8" x2="-165.1" y2="53.34" width="0.1524" layer="91"/>
+<wire x1="-165.1" y1="50.8" x2="-165.1" y2="48.26" width="0.1524" layer="91"/>
+<wire x1="-165.1" y1="48.26" x2="-165.1" y2="40.64" width="0.1524" layer="91"/>
+<wire x1="-165.1" y1="40.64" x2="-154.94" y2="40.64" width="0.1524" layer="91"/>
+<pinref part="C18" gate="G$1" pin="2"/>
+<pinref part="C17" gate="G$1" pin="2"/>
+<wire x1="-162.56" y1="48.26" x2="-165.1" y2="48.26" width="0.1524" layer="91"/>
+<pinref part="GND1" gate="1" pin="GND"/>
+<junction x="-165.1" y="63.5"/>
+<junction x="-165.1" y="60.96"/>
+<junction x="-165.1" y="58.42"/>
+<junction x="-165.1" y="55.88"/>
+<junction x="-165.1" y="53.34"/>
+<junction x="-165.1" y="50.8"/>
+<junction x="-165.1" y="48.26"/>
+<junction x="-144.78" y="58.42"/>
+<wire x1="-144.78" y1="58.42" x2="-144.78" y2="73.66" width="0.1524" layer="91"/>
+<label x="-144.78" y="73.66" size="1.27" layer="95" rot="R90" xref="yes"/>
+</segment>
+</net>

Commit message: Fixed TX pin disconnection
Signed-off-by: Bicoiu Ionut <159699747+bicoiu@users.noreply.github.com>
Connections:
- removed net N$5: TP1.TP
- net TX: now also TP1.TP
Changed lines of the file:
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@@
 </segment>
 <segment>
+<pinref part="TP1" gate="G$1" pin="TP"/>
+<wire x1="129.54" y1="71.12" x2="129.54" y2="73.66" width="0.1524" layer="91"/>
 <label x="129.54" y="73.66" size="1.27" layer="95" rot="R90" xref="yes"/>
 </segment>
@@
 </segment>
 </net>
-<net name="N$5" class="0">
-<segment>
-<pinref part="TP1" gate="G$1" pin="TP"/>
-<wire x1="129.54" y1="71.12" x2="129.54" y2="73.66" width="0.1524" layer="91"/>
-</segment>
-</net>
