File: Hardware/PCB.brd (EAGLE design)
At the start: 170.2 x 111.2 mm, 103 parts, among them IC1 BD5229G-TR, IC4 XC6220A331MR-G, J1 SAMACSYS_PARTS_USB4110-GF-A, J2 112A-TAAR-R03_ATTEND, J3 FH34SRJ-24S-0.5SH_99_, J4 QWIIC_RIGHT_ANGLE, Q1 20V/4.2A/52mΩ/1.4W, Q2 20V/4.2A/52mΩ/1.4W, Q3 SI1308EDL-T1-GE3, U1 W25Q512JVEIQ, U2 ESP32-C6-WROOM-1-N8, U3 DS3231SN#, U4 MAX17048G+T10

Commit message: Fixed 90 degree routes
Signed-off-by: Bicoiu Ionut <159699747+bicoiu@users.noreply.github.com>
Parts:
- removed MCP73831: ESP32_WROVER_SPARKFUN-IC-POWER_MCP73831, DeskAssistant v19 v1:ESP32_WROVER_SPARKFUN-IC-POWER_SOT23-5
- removed TP1, TP10, TP11, TP12, TP13, TP14, TP15, TP16, TP17, TP2, TP3, TP4, TP5, TP6, TP7, TP8, TP9: TPTP20R, DeskAssistant v19 v1:TP20R
- added 3V3, EPD_3V3, EPD_3V3_C, EPD_BUSY, EPD_CS, EPD_DC, EPD_RST, GND, GND_1, INT_RTC, MISO, MOSI, RX, SCK, TX, VBAT, VBUS: TPTP20R, DeskAssistant v19 v1:TP20R
- added U10: ESP32_WROVER_SPARKFUN-IC-POWER_MCP73831, DeskAssistant v19 v1:ESP32_WROVER_SPARKFUN-IC-POWER_SOT23-5
- C1: value 100nF -> 100uF
- C10, C2_BAT, C4, C5, C6, C7, C_DELAY, EPD_C1, EPD_C11, EPD_C12, EPD_C2, EPD_C6, EPD_C7, EPD_C8, EPD_C9: device DeskAssistant v19 v1:EAGLE-LTSPICE_C0402 -> DeskAssistant v19 v1:ESP32_WROVER_EAGLE-LTSPICE_C0402
- C3: value 100uF -> 100uF TANT
- C4_USB, C5_USB, C9: device DeskAssistant v19 v1:ESP32_WROVER_EAGLE-LTSPICE_C0402 -> DeskAssistant v19 v1:EAGLE-LTSPICE_C0402
- EPD_C10: value (none) -> 1uF/50V; device DeskAssistant v19 v1:EAGLE-LTSPICE_C0402 -> DeskAssistant v19 v1:ESP32_WROVER_EAGLE-LTSPICE_C0402
- EPD_C5: value 1uF/50V -> 0.1uF/50V; device DeskAssistant v19 v1:EAGLE-LTSPICE_C0402 -> DeskAssistant v19 v1:ESP32_WROVER_EAGLE-LTSPICE_C0402
- J1: value SAMACSYS_PARTS_USB4110-GF-A -> FH34SRJ-24S-0.5SH_99_; device DeskAssistant v19 v1:SAMACSYS_PARTS_USB4110GFA -> DeskAssistant v19 v1:FH34SRJ24S05SH99
- J2: value 112A-TAAR-R03_ATTEND -> SAMACSYS_PARTS_USB4110-GF-A; device DeskAssistant v19 v1:112ATAARR03ATTEND -> DeskAssistant v19 v1:SAMACSYS_PARTS_USB4110GFA
- J3: value FH34SRJ-24S-0.5SH_99_ -> QWIIC_RIGHT_ANGLE; device DeskAssistant v19 v1:FH34SRJ24S05SH99 -> DeskAssistant v19 v1:JST04_1MM_RA
- J4: value QWIIC_RIGHT_ANGLE -> 112A-TAAR-R03_ATTEND; device DeskAssistant v19 v1:JST04_1MM_RA -> DeskAssistant v19 v1:112ATAARR03ATTEND
- R10, R1_PINH, R1_PINH1, R2-PINH, R2-PINH1, R5, R6, R7, R8, R9, R_BOOT, R_CHANGE, R_CL1, R_RESET: value 10k -> 10K
- R2-USB: value 5k1 -> 5K1
- R2_BAT: value 2k -> 2K
- moved J4 184.0 mm to (6.05, 112.9), turned to 270 degrees
- moved J2 162.9 mm to (167.8, 71.3), turned to 90 degrees
- moved J3 84.4 mm to (165.3, 36.2), turned to 90 degrees
- moved J1 79.5 mm to (88.0, 29.5), turned to 0 degrees
- moved C2_BAT 31.9 mm to (128.0, 64.2)
- moved EPD_C2 28.3 mm to (92.4, 36.2), turned to 90 degrees
- moved EPD_C1 27.9 mm to (94.4, 36.1)
- moved L1 26.1 mm to (86.5, 63.7)
- moved D4 25.7 mm to (92.3, 55.9)
- moved R1_BAT 25.0 mm to (113.5, 63.1)
- moved C4 24.2 mm to (96.4, 59.6)
- moved D3 24.1 mm to (92.3, 59.4), turned to 180 degrees
- moved R1_PWRUSB 23.8 mm to (110.6, 51.2), turned to 270 degrees
- moved R_CL1 23.5 mm to (70.6, 56.2), turned to 270 degrees
- moved Q2 23.4 mm to (74.3, 56.2)
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Connections:
- removed net N$10: EPD_C2.2, J3.5
- removed net N$11: EPD_C12.2, J3.24
- removed net N$13: EPD_C10.2, J3.22
- removed net N$17: EPD_C6.2, J3.18
- removed net N$6 (its old number): MCP73831.1, R1_BAT.2
- removed net N$8 (its old number): MCP73831.5, R2_BAT.2
- new net N$19: EPD_C12.1, J1.24
- new net N$21: EPD_C10.1, J1.22
- new net N$23: EPD_C8.1, J1.20
- new net N$24: EPD_C7.1, J1.19
- new net N$25: EPD_C6.1, J1.18
- new net N$4: J2.A5, R2-USB1.2
- new net N$5: C1.1, C2.1
- new net RESE': R2.2, R3.1, SJ1.2
- net 3V3: now also 3V3.TP, J3.2, J4.P4; no longer J2.P4, J4.2, TP6.TP
- net DN: now also D1.4, J2.A7, J2.B7; no longer D1.6, J1.A7, J1.B7
- net DP: now also D1.6, J2.A6, J2.B6; no longer D1.4, J1.A6, J1.B6
- net EPD_3V3: now also EPD_3V3.TP, EPD_C5.1, J1.15, J1.16; no longer EPD_C5.2, J3.15, J3.16, TP7.TP
- net EPD_3V3_C: now also EPD_3V3_C.TP; no longer TP15.TP
- net EPD_BUSY: now also EPD_BUSY.TP, J1.9; no longer J3.9, TP8.TP
- net EPD_CS: now also EPD_CS.TP, J1.12; no longer J3.12, TP9.TP
- net EPD_DC: now also EPD_DC.TP, J1.11; no longer J3.11, TP13.TP
- net EPD_RST: now also EPD_RST.TP, J1.10; no longer J3.10, TP14.TP
- net GDR: now also J1.2; no longer J3.2
- net GND: now also EPD_C1.2, EPD_C10.2, EPD_C11.2, EPD_C12.2, EPD_C2.2, EPD_C5.2, EPD_C6.2, EPD_C7.2, EPD_C8.2, EPD_C9.2, GND.TP, GND_1.TP, J1.17, J1.8, J2.A1, J2.A12, J2.B1, J2.B12, J2.MP1, J2.MP2, J2.MP3, J2.MP4, J3.1, J4.G1, J4.G2, J4.G3, J4.G4, J4.P6, U10.2; no longer EPD_C1.1, EPD_C10.1, EPD_C11.1, EPD_C12.1, EPD_C2.1, EPD_C5.1, EPD_C6.1, EPD_C7.1, EPD_C8.1, EPD_C9.1, J1.A1, J1.A12, J1.B1, J1.B12, J1.MP3, J1.MP4, J2.G1, J2.G2, J2.G3, J2.G4, J2.P6, J3.17, J3.8, J3.MP1, J3.MP2, J4.1, MCP73831.2, TP4.TP, TP5.TP
- net I2C_PW: no longer C1.1, C2.1
- net INT_RTC: now also INT_RTC.TP; no longer TP17.TP
- net MISO: now also J4.P7, MISO.TP; no longer J2.P7, TP11.TP
- net MOSI: now also J1.14, J4.P3, MOSI.TP; no longer J2.P3, J3.14, TP12.TP
- net N$15: now also EPD_C2.1, J1.5; no longer EPD_C8.2, J3.20
- net N$16: now also EPD_C1.1, J1.4; no longer EPD_C7.2, J3.19
- net N$2: now also J2.B5; no longer J1.B5
- net N$3: now also R2_BAT.2, U10.5; no longer J1.A5, R2-USB1.2
- net N$9: now also R1_BAT.2, U10.1; no longer EPD_C1.2, J3.4
- net PREVGH: now also EPD_C9.1, J1.21; no longer EPD_C9.2, J3.21
- net PREVGL: now also EPD_C11.1, J1.23; no longer EPD_C11.2, J3.23
- net RESE: now also J1.3; no longer J3.3, R2.2, R3.1, SJ1.2
- net RX: now also RX.TP; no longer TP2.TP
- net SCK: now also J1.13, J4.P5, SCK.TP; no longer J2.P5, J3.13, TP10.TP
- net SCL: now also J3.4; no longer J4.4
- net SDA: now also J3.3; no longer J4.3
- net SS_SD: now also J4.P2; no longer J2.P2
- net TX: now also TX.TP; no longer TP1.TP
- net USB_D+: now also D1.1; no longer D1.3
- net USB_D-: now also D1.3; no longer D1.1
- net VBAT: now also U10.3, VBAT.TP; no longer MCP73831.3, TP3.TP
- net VBUS: now also U10.4, VBUS.TP; no longer MCP73831.4, TP16.TP
- net VUSB: now also J2.A4, J2.A9, J2.B4, J2.B9; no longer J1.A4, J1.A9, J1.B4, J1.B9
Routing:
- net TX: track 137.7 -> 4.44 mm, vias 2 -> 0
- net GND: track 834.5 -> 702.2 mm, vias 11 -> 10
- net VBUS: track 232.5 -> 107.3 mm, vias 4 -> 0
- net EPD_BUSY: track 227.2 -> 126.3 mm, vias 4 -> 5
- net RX: track 93.9 -> 4.78 mm, vias 2 -> 0
- net MISO: track 189.0 -> 111.6 mm, vias 4 -> 7
- net 3V3: track 536.2 -> 459.5 mm, vias 10 -> 8
- net SCK: track 252.3 -> 188.0 mm, vias 5 -> 6
- net INT_RTC: track 143.1 -> 92.3 mm, vias 2 -> 0
- net MOSI: track 238.9 -> 196.0 mm
- net VBAT: track 75.1 -> 33.4 mm, vias 2 -> 0
- net EPD_3V3: track 123.2 -> 81.6 mm, vias 5 -> 3
- net SDA: track 262.6 -> 226.0 mm, vias 4 -> 5
- net EPD_RST: track 159.2 -> 124.0 mm
- net N$10: track 29.8 -> 0.00 mm, vias 2 -> 0
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Other:
- board size 170.2 x 111.2 mm -> 170.2 x 111.4 mm

Commit message: Silkscreen Text overlapping
Signed-off-by: Bicoiu Ionut <159699747+bicoiu@users.noreply.github.com>
Parts:
- removed 3V3, EPD_3V3, EPD_3V3_C, EPD_BUSY, EPD_CS, EPD_DC, EPD_RST, GND, GND_1, INT_RTC, MISO, MOSI, RX, SCK, TX, VBAT, VBUS: TPTP20R, DeskAssistant v19 v1:TP20R
- removed U10: ESP32_WROVER_SPARKFUN-IC-POWER_MCP73831, DeskAssistant v19 v1:ESP32_WROVER_SPARKFUN-IC-POWER_SOT23-5
- added MCP73831: ESP32_WROVER_SPARKFUN-IC-POWER_MCP73831, DeskAssistant v19 v1:ESP32_WROVER_SPARKFUN-IC-POWER_SOT23-5
- added TP1, TP10, TP11, TP12, TP13, TP14, TP15, TP16, TP17, TP2, TP3, TP4, TP5, TP6, TP7, TP8, TP9: TPTP20R, DeskAssistant v19 v1:TP20R
- C1: value 100uF -> 100nF
- C10, C2_BAT, C4, C5, C6, C7, C_DELAY, EPD_C1, EPD_C11, EPD_C12, EPD_C2, EPD_C6, EPD_C7, EPD_C8, EPD_C9: device DeskAssistant v19 v1:ESP32_WROVER_EAGLE-LTSPICE_C0402 -> DeskAssistant v19 v1:EAGLE-LTSPICE_C0402
- C3: value 100uF TANT -> 100uF
- C4_USB, C5_USB, C9: device DeskAssistant v19 v1:EAGLE-LTSPICE_C0402 -> DeskAssistant v19 v1:ESP32_WROVER_EAGLE-LTSPICE_C0402
- EPD_C10: value 1uF/50V -> (none); device DeskAssistant v19 v1:ESP32_WROVER_EAGLE-LTSPICE_C0402 -> DeskAssistant v19 v1:EAGLE-LTSPICE_C0402
- EPD_C5: value 0.1uF/50V -> 1uF/50V; device DeskAssistant v19 v1:ESP32_WROVER_EAGLE-LTSPICE_C0402 -> DeskAssistant v19 v1:EAGLE-LTSPICE_C0402
- J1: value FH34SRJ-24S-0.5SH_99_ -> SAMACSYS_PARTS_USB4110-GF-A; device DeskAssistant v19 v1:FH34SRJ24S05SH99 -> DeskAssistant v19 v1:SAMACSYS_PARTS_USB4110GFA
- J2: value SAMACSYS_PARTS_USB4110-GF-A -> 112A-TAAR-R03_ATTEND; device DeskAssistant v19 v1:SAMACSYS_PARTS_USB4110GFA -> DeskAssistant v19 v1:112ATAARR03ATTEND
- J3: value QWIIC_RIGHT_ANGLE -> FH34SRJ-24S-0.5SH_99_; device DeskAssistant v19 v1:JST04_1MM_RA -> DeskAssistant v19 v1:FH34SRJ24S05SH99
- J4: value 112A-TAAR-R03_ATTEND -> QWIIC_RIGHT_ANGLE; device DeskAssistant v19 v1:112ATAARR03ATTEND -> DeskAssistant v19 v1:JST04_1MM_RA
- R10, R1_PINH, R1_PINH1, R2-PINH, R2-PINH1, R5, R6, R7, R8, R9, R_BOOT, R_CHANGE, R_CL1, R_RESET: value 10K -> 10k
- R2-USB: value 5K1 -> 5k1
- R2_BAT: value 2K -> 2k
- moved J4 184.0 mm to (164.4, 19.1), turned to 90 degrees
- moved J2 162.9 mm to (6.35, 92.7), turned to 270.4 degrees
- moved J3 84.4 mm to (83.8, 14.0), turned to 0 degrees
- moved J1 79.5 mm to (163.8, 53.3), turned to 90 degrees
- moved C2_BAT 31.9 mm to (116.8, 34.3)
- moved EPD_C2 28.3 mm to (69.8, 19.1), turned to 270 degrees
- moved EPD_C1 27.9 mm to (72.4, 19.1)
- moved L1 26.1 mm to (81.3, 38.1)
- moved D4 25.7 mm to (88.9, 30.5)
- moved R1_BAT 25.0 mm to (113.0, 38.1)
- moved C4 24.2 mm to (94.0, 35.6)
- moved D3 24.1 mm to (88.9, 35.6), turned to 0 degrees
- moved R1_PWRUSB 23.8 mm to (105.4, 27.9), turned to 90 degrees
- moved R_CL1 23.5 mm to (74.9, 33.0), turned to 90 degrees
- moved Q2 23.4 mm to (77.5, 33.0)
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Connections:
- removed net N$19: EPD_C12.1, J1.24
- removed net N$21: EPD_C10.1, J1.22
- removed net N$23: EPD_C8.1, J1.20
- removed net N$24: EPD_C7.1, J1.19
- removed net N$25: EPD_C6.1, J1.18
- removed net N$4 (its old number): J2.A5, R2-USB1.2
- removed net N$5 (its old number): C1.1, C2.1
- removed net RESE': R2.2, R3.1, SJ1.2
- new net N$10: EPD_C2.2, J3.5
- new net N$11: EPD_C12.2, J3.24
- new net N$13: EPD_C10.2, J3.22
- new net N$17: EPD_C6.2, J3.18
- new net N$6: MCP73831.1, R1_BAT.2
- new net N$8: MCP73831.5, R2_BAT.2
- net 3V3: now also J2.P4, J4.2, TP6.TP; no longer 3V3.TP, J3.2, J4.P4
- net DN: now also D1.6, J1.A7, J1.B7; no longer D1.4, J2.A7, J2.B7
- net DP: now also D1.4, J1.A6, J1.B6; no longer D1.6, J2.A6, J2.B6
- net EPD_3V3: now also EPD_C5.2, J3.15, J3.16, TP7.TP; no longer EPD_3V3.TP, EPD_C5.1, J1.15, J1.16
- net EPD_3V3_C: now also TP15.TP; no longer EPD_3V3_C.TP
- net EPD_BUSY: now also J3.9, TP8.TP; no longer EPD_BUSY.TP, J1.9
- net EPD_CS: now also J3.12, TP9.TP; no longer EPD_CS.TP, J1.12
- net EPD_DC: now also J3.11, TP13.TP; no longer EPD_DC.TP, J1.11
- net EPD_RST: now also J3.10, TP14.TP; no longer EPD_RST.TP, J1.10
- net GDR: now also J3.2; no longer J1.2
- net GND: now also EPD_C1.1, EPD_C10.1, EPD_C11.1, EPD_C12.1, EPD_C2.1, EPD_C5.1, EPD_C6.1, EPD_C7.1, EPD_C8.1, EPD_C9.1, J1.A1, J1.A12, J1.B1, J1.B12, J1.MP3, J1.MP4, J2.G1, J2.G2, J2.G3, J2.G4, J2.P6, J3.17, J3.8, J3.MP1, J3.MP2, J4.1, MCP73831.2, TP4.TP, TP5.TP; no longer EPD_C1.2, EPD_C10.2, EPD_C11.2, EPD_C12.2, EPD_C2.2, EPD_C5.2, EPD_C6.2, EPD_C7.2, EPD_C8.2, EPD_C9.2, GND.TP, GND_1.TP, J1.17, J1.8, J2.A1, J2.A12, J2.B1, J2.B12, J2.MP1, J2.MP2, J2.MP3, J2.MP4, J3.1, J4.G1, J4.G2, J4.G3, J4.G4, J4.P6, U10.2
- net I2C_PW: now also C1.1, C2.1
- net INT_RTC: now also TP17.TP; no longer INT_RTC.TP
- net MISO: now also J2.P7, TP11.TP; no longer J4.P7, MISO.TP
- net MOSI: now also J2.P3, J3.14, TP12.TP; no longer J1.14, J4.P3, MOSI.TP
- net N$15: now also EPD_C8.2, J3.20; no longer EPD_C2.1, J1.5
- net N$16: now also EPD_C7.2, J3.19; no longer EPD_C1.1, J1.4
- net N$2: now also J1.B5; no longer J2.B5
- net N$3: now also J1.A5, R2-USB1.2; no longer R2_BAT.2, U10.5
- net N$9: now also EPD_C1.2, J3.4; no longer R1_BAT.2, U10.1
- net PREVGH: now also EPD_C9.2, J3.21; no longer EPD_C9.1, J1.21
- net PREVGL: now also EPD_C11.2, J3.23; no longer EPD_C11.1, J1.23
- net RESE: now also J3.3, R2.2, R3.1, SJ1.2; no longer J1.3
- net RX: now also TP2.TP; no longer RX.TP
- net SCK: now also J2.P5, J3.13, TP10.TP; no longer J1.13, J4.P5, SCK.TP
- net SCL: now also J4.4; no longer J3.4
- net SDA: now also J4.3; no longer J3.3
- net SS_SD: now also J2.P2; no longer J4.P2
- net TX: now also TP1.TP; no longer TX.TP
- net USB_D+: now also D1.3; no longer D1.1
- net USB_D-: now also D1.1; no longer D1.3
- net VBAT: now also MCP73831.3, TP3.TP; no longer U10.3, VBAT.TP
- net VBUS: now also MCP73831.4, TP16.TP; no longer U10.4, VBUS.TP
- net VUSB: now also J1.A4, J1.A9, J1.B4, J1.B9; no longer J2.A4, J2.A9, J2.B4, J2.B9
Routing:
- net TX: track 4.44 -> 137.7 mm, vias 0 -> 2
- net VBUS: track 107.3 -> 233.1 mm, vias 0 -> 4
- net GND: track 702.2 -> 827.8 mm, vias 10 -> 11
- net EPD_BUSY: track 126.3 -> 229.2 mm, vias 5 -> 4
- net RX: track 4.78 -> 93.9 mm, vias 0 -> 2
- net 3V3: track 459.5 -> 542.9 mm, vias 8 -> 10
- net MISO: track 111.6 -> 186.8 mm, vias 7 -> 4
- net SCK: track 188.0 -> 252.7 mm, vias 6 -> 5
- net MOSI: track 196.0 -> 242.3 mm
- net INT_RTC: track 92.3 -> 137.0 mm, vias 0 -> 2
- net VBAT: track 33.4 -> 75.1 mm, vias 0 -> 2
- net EPD_3V3: track 81.6 -> 119.0 mm, vias 3 -> 5
- net EPD_RST: track 124.0 -> 156.9 mm
- net SDA: track 226.0 -> 256.4 mm, vias 5 -> 4
- net SS_SD: track 71.4 -> 101.6 mm, vias 0 -> 3
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Other:
- board size 170.2 x 111.4 mm -> 170.2 x 111.2 mm
